File: AS5048B/AS5048B.kicad_sch (KiCad schematic)
At the start: 5 parts, among them J1 Conn_01x04_Socket, Q1 AS5048B-HTSP-500

Commit message: Updated Logo
Parts:
- C1: footprint Capacitor_SMD:C_0603_1608Metric_Pad1.08x0.95mm_HandSolder -> Capacitor_SMD:C_0603_1608Metric; Comment (none) -> 10uF, X5R 6.3V; LCSC Part Number (none) -> C95839
- C2: footprint Capacitor_SMD:C_0603_1608Metric_Pad1.08x0.95mm_HandSolder -> Capacitor_SMD:C_0603_1608Metric; Comment (none) -> 100nF, X7R 16V; LCSC Part Number (none) -> C66501
- J1: Comment (none) -> JST GH SM04B; LCSC Part Number (none) -> C189895
- JP1: Comment (none) -> Not Placed
Changed lines of the file:
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@@
+			)
+		)
+		(property "Comment" "Not Placed"
+			(at 100.33 73.66 0)
+			(effects
+				(font
+					(size 1.27 1.27)
+				)
+				(hide yes)
+			)
+		)
+		(property "LCSC Part Number" ""
+			(at 100.33 73.66 0)
+			(effects
+				(font
+					(size 1.27 1.27)
+				)
+				(hide yes)
 			)
 		)
@@
 			)
 		)
-		(property "Footprint" "Capacitor_SMD:C_0603_1608Metric_Pad1.08x0.95mm_HandSolder"
+		(property "Footprint" "Capacitor_SMD:C_0603_1608Metric"
 			(at 152.4 102.5652 0)
 			(effects
@@
 			)
 		)
+		(property "Comment" "10uF, X5R 6.3V"
+			(at 156.21 101.6 0)
+			(effects
+				(font
+					(size 1.27 1.27)
+				)
+				(hide yes)
+			)
+		)
+		(property "LCSC Part Number" "C95839"
+			(at 156.21 101.6 0)
+			(effects
+				(font
+					(size 1.27 1.27)
+				)
+				(hide yes)
+			)
+		)
 		(pin "1"
 		)
@@
 			)
 		)
-		(property "Footprint" "Capacitor_SMD:C_0603_1608Metric_Pad1.08x0.95mm_HandSolder"
+		(property "Footprint" "Capacitor_SMD:C_0603_1608Metric"
 			(at 160.02 113.3348 0)
 			(effects
@@
 			)
 		)
+		(property "Comment" "100nF, X7R 16V"
+			(at 156.21 114.3 0)
+			(effects
+				(font
+					(size 1.27 1.27)
+				)
+				(hide yes)
+			)
+		)
+		(property "LCSC Part Number" "C66501"
+			(at 156.21 114.3 0)
+			(effects
+				(font
+					(size 1.27 1.27)
+				)
+				(hide yes)
+			)
+		)
 		(pin "1"
 		)
@@
 			)
 		)
-		(property "Datasheet" "AS5048B-HTSP-500"
+		(property "Datasheet" "https://www.mouser.com/datasheet/2/588/AS5048_DS000298_4_00-2324531.pdf"
 			(at 104.14 90.17 0)
 			(effects
@@
 		)
 		(property "Description" ""
+			(at 104.14 90.17 0)
+			(effects
+				(font
+					(size 1.27 1.27)
+				)
+				(hide yes)
+			)
+		)
+		(property "Comment" ""
+			(at 104.14 90.17 0)
+			(effects
+				(font
+					(size 1.27 1.27)
+				)
+				(hide yes)
+			)
+		)
+		(property "LCSC Part Number" ""
 			(at 104.14 90.17 0)
 			(effects
@@
 			(at 88.9 63.5 0)
 			(effects
+				(font
+					(size 1.27 1.27)
+				)
+				(hide yes)
+			)
+		)
+		(property "Comment" "JST GH SM04B"
+			(at 88.9 63.5 0)
+			(effects
+				(font
+					(size 1.27 1.27)
+				)
+				(hide yes)
+			)
+		)
+		(property "LCSC Part Number" "C189895"
+			(at 88.9 63.5 0)
+			(effects
