File: MT6701/MT6701.kicad_pcb (KiCad board)
At the start: 2 copper layers, 23.2 x 23.2 mm, 7 parts, among them Q1 AS5048B-HTSP-500

Commit message: Updated Schematic
Parts:
- removed C1: 10uF, Capacitor_SMD:C_0603_1608Metric
- removed C2: 100nF, Capacitor_SMD:C_0603_1608Metric
- removed G***: LOGO, Sharkbite:Logo1 8x8
- removed JP1: SolderJumper_3_Open, Jumper:SolderJumper-3_P1.3mm_Open_RoundedPad1.0x1.5mm
- removed Je: Conn_01x04_Socket, Connector_JST:JST_GH_SM04B-GHS-TB_1x04-1MP_P1.25mm_Horizontal
- removed Q1: AS5048B-HTSP-500, Ethan:TRANS_HTSP-500_AMS
- removed REF**: 18XX-20XX Motor, Library:Slot
- added D1: SMAJ6.0A, Diode_SMD:D_SMA, F.Cu at (124.2, 146.0)
- added J1: Conn_01x05_Pin, Connector_JST:JST_GH_SM05B-GHS-TB_1x05-1MP_P1.25mm_Horizontal, F.Cu at (126.0, 140.0)
- added U1: MT6701QT, Package_DFN_QFN:QFN-16-1EP_3x3mm_P0.5mm_EP1.7x1.7mm, F.Cu at (130.9, 146.4)
Routing:
- net +5V: track 20.2 -> 0.00 mm, vias 2 -> 0
- net Net-(J1-Pin_4): track 18.5 -> 0.00 mm, vias 2 -> 0
- net /PWM: track 15.0 -> 0.00 mm, vias 1 -> 0
- net GND: track 15.7 -> 0.81 mm, vias 7 -> 5
- net /I2C: track 12.1 -> 0.00 mm, vias 1 -> 0
- net Net-(Q1-VDD3V): track 11.4 -> 0.00 mm, vias 1 -> 0
- net Net-(J1-Pin_3): track 9.25 -> 0.00 mm, vias 1 -> 0

Commit message: V1 Order
Parts:
- removed D1: SMAJ6.0A, Diode_SMD:D_SMA
- added C1: 100nF, Capacitor_SMD:C_0402_1005Metric, F.Cu at (150.0, 147.4)
- added G***: LOGO, Sharkbite:Logo1 8x8, B.Cu at (149.3, 150.2)
- added JP1: SolderJumper_2_Open, Jumper:SolderJumper-2_P1.3mm_Open_TrianglePad1.0x1.5mm, B.Cu at (154.7, 145.3)
- added R1: 5K, Resistor_SMD:R_0402_1005Metric, F.Cu at (152.6, 150.1)
- added R2: 5K, Resistor_SMD:R_0402_1005Metric, F.Cu at (147.4, 150.0)
- added REF**: 18XX-20XX Motor, Sharkbite:18XX-20XX Motor, F.Cu at (150.0, 150.1)
- added TP1: TestPoint, TestPoint:TestPoint_Pad_1.0x1.0mm, B.Cu at (146.5, 156.4)
- J1: moved to B.Cu
- moved U1 19.4 mm to (150.0, 150.0)
- moved J1 17.9 mm to (143.6, 143.6), turned to 45 degrees
Connections:
- J1 pad MP: (no net) -> GND
- U1 pad 15: Net-(U1-OUT) -> unconnected-(U1-OUT-Pad15)
Routing:
- net +5V: track 0.00 -> 20.8 mm, vias 0 -> 2
- net /VDD/CSN: track 0.00 -> 20.1 mm, vias 0 -> 1
- net /SCL/CLK: track 0.00 -> 17.0 mm, vias 0 -> 3
- net /SDA/DO: track 0.00 -> 16.8 mm, vias 0 -> 1
- net Net-(U1-PUSH): track 0.00 -> 6.74 mm, vias 0 -> 1
- net GND: track 0.81 -> 1.25 mm, vias 5 -> 9
Other:
- board text removed: "I2C"
- board text removed: "PWM"
